File: pcb/RPi-Proto-HAT_v10.sch (EAGLE design)
At the start: 36 parts, among them X1 PASSER-07, X2 PASSER-07

Commit message: cleaned up schematics and layout
Other:
- note removed: "www.watterott.com"
Changed lines of the file:
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@@
 <setting verticaltext="up"/>
 </settings>
-<grid distance="0.1" unitdist="inch" unit="inch" style="lines" multiple="1" display="no" altdistance="0.01" altunitdist="inch" altunit="inch"/>
+<grid distance="0.05" unitdist="inch" unit="inch" style="lines" multiple="1" display="yes" altdistance="0.025" altunitdist="inch" altunit="inch"/>
 <layers>
 <layer number="1" name="Top" color="4" fill="1" visible="no" active="no"/>
@@
 </classes>
 <parts>
-<part name="FRAME1" library="frames" deviceset="A4L-LOC" device=""/>
 <part name="P+2" library="supply1" deviceset="+5V" device=""/>
 <part name="GND4" library="supply1" deviceset="GND" device=""/>
@@
 <part name="15" library="we-rcl" deviceset="PAD" device="-1-1.6"/>
 <part name="14" library="we-rcl" deviceset="PAD" device="-1-1.6"/>
+<part name="FRAME1" library="we-symbol" deviceset="FRAME-A4L" device=""/>
 </parts>
 <sheets>
@@
 <plain>
 <text x="52.07" y="130.81" size="3.81" layer="250">Raspberry Pi B+</text>
-<text x="161.29" y="31.75" size="1.27" layer="95">Released under the Creative Commons Attribution Share-Alike License</text>
-<text x="161.29" y="29.21" size="1.27" layer="95">http://creativecommons.org/licenses/by-sa/4.0/</text>
-<text x="161.29" y="25.4" size="1.27" layer="95">Designed by Andreas Watterott (Watterott electronic)</text>
+<text x="162.56" y="21.59" size="1.27" layer="95">Released under the Creative Commons Attribution Share-Alike License</text>
+<text x="162.56" y="19.05" size="1.27" layer="95">http://creativecommons.org/licenses/by-sa/4.0/</text>
+<text x="162.56" y="15.24" size="1.27" layer="95">Designed by Andreas Watterott (Watterott electronic)</text>
 <text x="152.4" y="130.81" size="3.81" layer="250">ID EEPROM</text>
 <text x="147.32" y="125.73" size="1.27" layer="250" font="vector">OnSemi CAT24C32 or Microchip 24LC32A</text>
-<text x="213.36" y="5.08" size="2.54" layer="94" font="vector" align="bottom-right">www.watterott.com</text>
 </plain>
 <instances>
-<instance part="FRAME1" gate="G$1" x="0" y="0" smashed="yes">
-<attribute name="DRAWING_NAME" x="217.17" y="15.24" size="2.54" layer="94" font="vector"/>
-<attribute name="LAST_DATE_TIME" x="217.17" y="10.16" size="2.286" layer="94" font="vector"/>
-<attribute name="SHEET" x="230.505" y="5.08" size="2.54" layer="94" font="vector"/>
-</instance>
 <instance part="P+2" gate="1" x="90.17" y="119.38" smashed="yes" rot="R270">
 <attribute name="VALUE" x="92.71" y="117.475" size="1.778" layer="96" rot="R90"/>
@@
 <instance part="R2" gate="R" x="191.77" y="111.76" rot="R90"/>
 <instance part="R3" gate="R" x="151.13" y="107.95" rot="R90"/>
-<instance part="X1" gate="X" x="166.37" y="19.05"/>
-<instance part="X2" gate="X" x="173.99" y="19.05"/>
-<instance part="LOGO2" gate="G$1" x="207.01" y="19.05"/>
+<instance part="X1" gate="X" x="165.1" y="7.62"/>
+<instance part="X2" gate="X" x="170.18" y="7.62"/>
+<instance part="LOGO2" gate="G$1" x="208.28" y="7.62"/>
 <instance part="IC" gate="IC" x="168.91" y="106.68"/>
 <instance part="2" gate="X" x="41.91" y="118.11"/>
@@
 <instance part="15" gate="X" x="97.79" y="110.49" rot="R180"/>
 <instance part="14" gate="X" x="97.79" y="113.03" rot="R180"/>
+<instance part="FRAME1" gate="G$1" x="0" y="0"/>
 </instances>
 <busses>
